File: REF1190.kicad_pcb (KiCad board)
At the start: 2 copper layers, 101.7 x 58.1 mm, 19 parts, among them J1 DNP, J2 DNP, J3 DNP, J4 DNP, J5 DNP, J6 DNP, J7 Jumper 2, J8 Jumper 1, J9 DB25_Pins_MountingHoles, U2 74HC373, U3 74HC373, U4 74HC74

Commit message: Add files via upload
Parts:
- renumbered R3 to D1
Changed lines of the file:
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@@
 		(layer "F.Cu")
 		(at 114.629 63.204)
-		(property "Reference" "R3"
+		(property "Reference" "D1"
 			(at 4 0 0)
 			(layer "F.SilkS")
@@
 			(stroke
 				(width 0.12)
-				(type default)
-			)
-			(layer "F.SilkS")
-		)
-		(fp_line
-			(start 2.8 -1.3)
-			(end 2.8 1.3)
-			(stroke
-				(width 0.12)
